Commit message: Removed unused red material declaration.

File: reemc_common/reemc_description/urdf/sensors/mvbluefox_camera.urdf.xacro (robot description, xacro)
@@ -33,7 +33,4 @@
         <material name="Blue" />
       </visual>
-      <material name="Red">
-        <color rgba="0.72941 0.35686 0.023529 1" />
-      </material>
     </link>
   </xacro:macro>

File: reemc_common/reemc_description/urdf/sensors/prosilicaGC655C_camera.urdf.xacro (robot description, xacro)
@@ -33,7 +33,4 @@
         <material name="Blue" />
       </visual>
-      <material name="Red">
-        <color rgba="0.72941 0.35686 0.023529 1" />
-      </material>
     </link>
   </xacro:macro>
