Commit message: Removed unused xml namespaces.

File: reemc_common/reemc_description/urdf/arm/arm.transmission.xacro (robot description, xacro)
@@ -7,8 +7,5 @@
   Creative Commons, 444 Castro Street, Suite 900, Mountain View, California, 94041, USA.
 -->
-<robot xmlns:sensor="http://playerstage.sourceforge.net/gazebo/xmlschema/#sensor"
-       xmlns:controller="http://playerstage.sourceforge.net/gazebo/xmlschema/#controller"
-       xmlns:interface="http://playerstage.sourceforge.net/gazebo/xmlschema/#interface"
-       xmlns:xacro="http://ros.org/wiki/xacro">
+<robot xmlns:xacro="http://ros.org/wiki/xacro">
   <xacro:macro name="reem_arm_simple_transmission" params="name side number reduction" >
     <transmission name="${name}_${side}_${number}_trans">

File: reemc_common/reemc_description/urdf/arm/arm.urdf.xacro (robot description, xacro)
@@ -7,8 +7,5 @@
   Creative Commons, 444 Castro Street, Suite 900, Mountain View, California, 94041, USA.
 -->
-<robot xmlns:sensor="http://playerstage.sourceforge.net/gazebo/xmlschema/#sensor"
-       xmlns:controller="http://playerstage.sourceforge.net/gazebo/xmlschema/#controller"
-       xmlns:interface="http://playerstage.sourceforge.net/gazebo/xmlschema/#interface"
-       xmlns:xacro="http://ros.org/wiki/xacro">
+<robot xmlns:xacro="http://ros.org/wiki/xacro">
   <!--File includes-->
   <include filename="$(find reemc_description)/urdf/deg_to_rad.xacro" />

File: reemc_common/reemc_description/urdf/arm/wrist.transmission.xacro (robot description, xacro)
@@ -7,8 +7,5 @@
   Creative Commons, 444 Castro Street, Suite 900, Mountain View, California, 94041, USA.
 -->
-<robot xmlns:sensor="http://playerstage.sourceforge.net/gazebo/xmlschema/#sensor"
-       xmlns:controller="http://playerstage.sourceforge.net/gazebo/xmlschema/#controller"
-       xmlns:interface="http://playerstage.sourceforge.net/gazebo/xmlschema/#interface"
-       xmlns:xacro="http://ros.org/wiki/xacro">
+<robot xmlns:xacro="http://ros.org/wiki/xacro">
   <xacro:macro name="reem_wrist_simple_transmission" params="name side number reduction" >
     <transmission name="${name}_${side}_${number}_trans">

File: reemc_common/reemc_description/urdf/arm/wrist.urdf.xacro (robot description, xacro)
@@ -7,8 +7,5 @@
   Creative Commons, 444 Castro Street, Suite 900, Mountain View, California, 94041, USA.
 -->
-<robot xmlns:sensor="http://playerstage.sourceforge.net/gazebo/xmlschema/#sensor"
-       xmlns:controller="http://playerstage.sourceforge.net/gazebo/xmlschema/#controller"
-       xmlns:interface="http://playerstage.sourceforge.net/gazebo/xmlschema/#interface"
-       xmlns:xacro="http://ros.org/wiki/xacro">
+<robot xmlns:xacro="http://ros.org/wiki/xacro">
   <!--File includes-->
   <include filename="$(find reemc_description)/urdf/deg_to_rad.xacro" />

File: reemc_common/reemc_description/urdf/foot/foot.urdf.xacro (robot description, xacro)
@@ -7,8 +7,5 @@
   Creative Commons, 444 Castro Street, Suite 900, Mountain View, California, 94041, USA.
 -->
-<robot name="reemc" xmlns:sensor="http://playerstage.sourceforge.net/gazebo/xmlschema/#sensor"
-       xmlns:controller="http://playerstage.sourceforge.net/gazebo/xmlschema/#controller"
-       xmlns:interface="http://playerstage.sourceforge.net/gazebo/xmlschema/#interface"
-       xmlns:xacro="http://ros.org/wiki/xacro">
+<robot name="reemc" xmlns:xacro="http://ros.org/wiki/xacro">
   <xacro:macro name="reemc_foot" params="name parent side reflect">
     <link name="r_foot">

File: reemc_common/reemc_description/urdf/hand/hand.gazebo.xacro (robot description, xacro)
@@ -7,8 +7,5 @@
   Creative Commons, 444 Castro Street, Suite 900, Mountain View, California, 94041, USA.
 -->
-<robot xmlns:sensor="http://playerstage.sourceforge.net/gazebo/xmlschema/#sensor"
-       xmlns:controller="http://playerstage.sourceforge.net/gazebo/xmlschema/#controller"
-       xmlns:interface="http://playerstage.sourceforge.net/gazebo/xmlschema/#interface"
-       xmlns:xacro="http://ros.org/wiki/xacro">
+<robot xmlns:xacro="http://ros.org/wiki/xacro">
     <xacro:macro name="hand_grasping_hack" params="side">
       <gazebo>

File: reemc_common/reemc_description/urdf/hand/hand.transmission.xacro (robot description, xacro)
@@ -7,8 +7,5 @@
   Creative Commons, 444 Castro Street, Suite 900, Mountain View, California, 94041, USA.
 -->
-<robot xmlns:sensor="http://playerstage.sourceforge.net/gazebo/xmlschema/#sensor"
-      xmlns:controller="http://playerstage.sourceforge.net/gazebo/xmlschema/#controller"
-      xmlns:interface="http://playerstage.sourceforge.net/gazebo/xmlschema/#interface"
-      xmlns:xacro="http://ros.org/wiki/xacro">
+<robot xmlns:xacro="http://ros.org/wiki/xacro">
  <!-- Thumb -->
   <xacro:macro name="hand_thumb_transmission" params="name reduction" >

File: reemc_common/reemc_description/urdf/hand/hand.urdf.xacro (robot description, xacro)
@@ -7,8 +7,5 @@
   Creative Commons, 444 Castro Street, Suite 900, Mountain View, California, 94041, USA.
 -->
-<robot xmlns:sensor="http://playerstage.sourceforge.net/gazebo/xmlschema/#sensor"
-      xmlns:controller="http://playerstage.sourceforge.net/gazebo/xmlschema/#controller"
-      xmlns:interface="http://playerstage.sourceforge.net/gazebo/xmlschema/#interface"
-      xmlns:xacro="http://ros.org/wiki/xacro">
+<robot xmlns:xacro="http://ros.org/wiki/xacro">
   <!--File includes-->
   <include filename="$(find reemc_description)/urdf/deg_to_rad.xacro" />

File: reemc_common/reemc_description/urdf/head/head.transmission.xacro (robot description, xacro)
@@ -7,8 +7,5 @@
   Creative Commons, 444 Castro Street, Suite 900, Mountain View, California, 94041, USA.
 -->
-<robot xmlns:sensor="http://playerstage.sourceforge.net/gazebo/xmlschema/#sensor"
-       xmlns:controller="http://playerstage.sourceforge.net/gazebo/xmlschema/#controller"
-       xmlns:interface="http://playerstage.sourceforge.net/gazebo/xmlschema/#interface"
-       xmlns:xacro="http://ros.org/wiki/xacro">
+<robot xmlns:xacro="http://ros.org/wiki/xacro">
   <xacro:macro name="head_transmission" params="name reduction">
     <transmission name="${name}_trans">

File: reemc_common/reemc_description/urdf/head/head.urdf.xacro (robot description, xacro)
@@ -7,8 +7,5 @@
   Creative Commons, 444 Castro Street, Suite 900, Mountain View, California, 94041, USA.
 -->
-<robot xmlns:sensor="http://playerstage.sourceforge.net/gazebo/xmlschema/#sensor"
-       xmlns:controller="http://playerstage.sourceforge.net/gazebo/xmlschema/#controller"
-       xmlns:interface="http://playerstage.sourceforge.net/gazebo/xmlschema/#interface"
-       xmlns:xacro="http://ros.org/wiki/xacro">
+<robot xmlns:xacro="http://ros.org/wiki/xacro">
   <!--File includes-->
   <include filename="$(find reemc_description)/urdf/deg_to_rad.xacro" />

File: reemc_common/reemc_description/urdf/leg/leg.transmission.xacro (robot description, xacro)
@@ -7,8 +7,5 @@
   Creative Commons, 444 Castro Street, Suite 900, Mountain View, California, 94041, USA.
 -->
-<robot name="reemc" xmlns:sensor="http://playerstage.sourceforge.net/gazebo/xmlschema/#sensor"
-       xmlns:controller="http://playerstage.sourceforge.net/gazebo/xmlschema/#controller"
-       xmlns:interface="http://playerstage.sourceforge.net/gazebo/xmlschema/#interface"
-       xmlns:xacro="http://ros.org/wiki/xacro">
+<robot name="reemc" xmlns:xacro="http://ros.org/wiki/xacro">
   <xacro:macro name="reemc_leg_simple_transmission" params="name side number reduction" >
     <transmission name="${name}_${side}_${number}_trans">

File: reemc_common/reemc_description/urdf/leg/leg.urdf.xacro (robot description, xacro)
@@ -7,8 +7,5 @@
   Creative Commons, 444 Castro Street, Suite 900, Mountain View, California, 94041, USA.
 -->
-<robot name="reemc" xmlns:sensor="http://playerstage.sourceforge.net/gazebo/xmlschema/#sensor"
-       xmlns:controller="http://playerstage.sourceforge.net/gazebo/xmlschema/#controller"
-       xmlns:interface="http://playerstage.sourceforge.net/gazebo/xmlschema/#interface"
-       xmlns:xacro="http://ros.org/wiki/xacro">
+<robot name="reemc" xmlns:xacro="http://ros.org/wiki/xacro">
   <!--File includes-->
   <include filename="$(find reemc_description)/urdf/deg_to_rad.xacro" />

File: reemc_common/reemc_description/urdf/sensors/back_camera.urdf.xacro (robot description, xacro)
@@ -7,8 +7,5 @@
   Creative Commons, 444 Castro Street, Suite 900, Mountain View, California, 94041, USA.
 -->
-<robot xmlns:sensor="http://playerstage.sourceforge.net/gazebo/xmlschema/#sensor"
-       xmlns:controller="http://playerstage.sourceforge.net/gazebo/xmlschema/#controller"
-       xmlns:interface="http://playerstage.sourceforge.net/gazebo/xmlschema/#interface"
-       xmlns:xacro="http://ros.org/wiki/xacro">
+<robot xmlns:xacro="http://ros.org/wiki/xacro">
   <!-- back camera macro uses stingrayf033c_camera macros -->
   <include filename="$(find reemc_description)/urdf/sensors/mvbluefox_back_camera.gazebo.xacro" />

File: reemc_common/reemc_description/urdf/sensors/ftsensor.gazebo.xacro (robot description, xacro)
@@ -7,8 +7,5 @@
   Creative Commons, 444 Castro Street, Suite 900, Mountain View, California, 94041, USA.
 -->
-<robot name="reemc" xmlns:sensor="http://playerstage.sourceforge.net/gazebo/xmlschema/#sensor"
-       xmlns:controller="http://playerstage.sourceforge.net/gazebo/xmlschema/#controller"
-       xmlns:interface="http://playerstage.sourceforge.net/gazebo/xmlschema/#interface"
-       xmlns:xacro="http://ros.org/wiki/xacro">
+<robot name="reemc" xmlns:xacro="http://ros.org/wiki/xacro">
 <xacro:macro name="reemc_force_torque_sensor" params="name update_rate">
   <gazebo reference="${name}">

File: reemc_common/reemc_description/urdf/sensors/imu.urdf.xacro (robot description, xacro)
@@ -7,8 +7,5 @@
   Creative Commons, 444 Castro Street, Suite 900, Mountain View, California, 94041, USA.
 -->
-<robot name="reemc" xmlns:sensor="http://playerstage.sourceforge.net/gazebo/xmlschema/#sensor"
-       xmlns:controller="http://playerstage.sourceforge.net/gazebo/xmlschema/#controller"
-       xmlns:interface="http://playerstage.sourceforge.net/gazebo/xmlschema/#interface"
-       xmlns:xacro="http://ros.org/wiki/xacro">
+<robot name="reemc" xmlns:xacro="http://ros.org/wiki/xacro">
   <xacro:macro name="reemc_imu" params="name parent update_rate">
     <link name="${name}_link">

File: reemc_common/reemc_description/urdf/sensors/laser.urdf.xacro (robot description, xacro)
@@ -7,8 +7,5 @@
   Creative Commons, 444 Castro Street, Suite 900, Mountain View, California, 94041, USA.
 -->
-<robot xmlns:sensor="http://playerstage.sourceforge.net/gazebo/xmlschema/#sensor"
-      xmlns:controller="http://playerstage.sourceforge.net/gazebo/xmlschema/#controller"
-      xmlns:interface="http://playerstage.sourceforge.net/gazebo/xmlschema/#interface"
-      xmlns:xacro="http://ros.org/wiki/xacro">
+<robot xmlns:xacro="http://ros.org/wiki/xacro">
   <include filename="$(find reemc_description)/urdf/sensors/laser.gazebo.xacro" />
   <xacro:macro name="reemc_laser" params="name parent *origin ros_topic update_rate min_angle max_angle nrays">

File: reemc_common/reemc_description/urdf/sensors/mvbluefox_camera.urdf.xacro (robot description, xacro)
@@ -8,8 +8,5 @@
 -->
 <!-- XML namespaces -->
-<robot name="reemc" xmlns:sensor="http://playerstage.sourceforge.net/gazebo/xmlschema/#sensor"
-       xmlns:controller="http://playerstage.sourceforge.net/gazebo/xmlschema/#controller"
-       xmlns:interface="http://playerstage.sourceforge.net/gazebo/xmlschema/#interface"
-       xmlns:xacro="http://ros.org/wiki/xacro">
+<robot name="reemc" xmlns:xacro="http://ros.org/wiki/xacro">
   <xacro:macro name="mvbluefox_camera" params="name parent *origin">
     <joint name="${name}_frame_joint" type="fixed">
@@ -31,5 +28,5 @@
           <cylinder radius="0.01" length="0.02" />
         </geometry>
-        <material name="Blue" />
+        <material name="Blue"/>
       </visual>
     </link>

File: reemc_common/reemc_description/urdf/sensors/openni.gazebo.xacro (robot description, xacro)
@@ -11,8 +11,5 @@
   Sensor parameters are from PR2 description.
 -->
-<robot xmlns:sensor="http://playerstage.sourceforge.net/gazebo/xmlschema/#sensor"
-       xmlns:controller="http://playerstage.sourceforge.net/gazebo/xmlschema/#controller"
-       xmlns:interface="http://playerstage.sourceforge.net/gazebo/xmlschema/#interface"
-       xmlns:xacro="http://ros.org/wiki/xacro">
+<robot xmlns:xacro="http://ros.org/wiki/xacro">
   <xacro:macro name="openni_ir_gazebo_v0" params="link_name frame_name camera_name">
     <gazebo reference="${link_name}">

File: reemc_common/reemc_description/urdf/sensors/prosilicaGC655C_camera.urdf.xacro (robot description, xacro)
@@ -8,8 +8,5 @@
 -->
 <!-- XML namespaces -->
-<robot name="reemc" xmlns:sensor="http://playerstage.sourceforge.net/gazebo/xmlschema/#sensor"
-       xmlns:controller="http://playerstage.sourceforge.net/gazebo/xmlschema/#controller"
-       xmlns:interface="http://playerstage.sourceforge.net/gazebo/xmlschema/#interface"
-       xmlns:xacro="http://ros.org/wiki/xacro">
+<robot name="reemc" xmlns:xacro="http://www.ros.org/wiki/xacro">
   <xacro:macro name="prosilicaGC655C_camera" params="name parent *origin">
     <joint name="${name}_frame_joint" type="fixed">
@@ -31,5 +28,5 @@
           <cylinder radius="0.01" length="0.018" />
         </geometry>
-        <material name="Blue" />
+        <material name="Blue"/>
       </visual>
     </link>

File: reemc_common/reemc_description/urdf/sensors/prosilica_stereo_camera.gazebo.xacro (robot description, xacro)
@@ -7,8 +7,5 @@
   Creative Commons, 444 Castro Street, Suite 900, Mountain View, California, 94041, USA.
 -->
-<robot name="reemc" xmlns:sensor="http://playerstage.sourceforge.net/gazebo/xmlschema/#sensor"
-       xmlns:controller="http://playerstage.sourceforge.net/gazebo/xmlschema/#controller"
-       xmlns:interface="http://playerstage.sourceforge.net/gazebo/xmlschema/#interface"
-       xmlns:xacro="http://ros.org/wiki/xacro">
+<robot name="reemc" xmlns:xacro="http://ros.org/wiki/xacro">
   <xacro:macro name="prosilica_stereo_camera_gazebo" params="name image_format hfov focal_length frame_id hack_baseline image_width image_height">
     <gazebo reference="${name}_link">
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