Commit message: Replaced meshes with updated versions in dae format. Updated urdf files accordingly.

File: reemc_common/reemc_description/robots/reemc_full.urdf.xacro (robot description, xacro)
@@ -20,5 +20,5 @@
       <origin rpy="0 0 0" xyz="0 0 0"/>
       <geometry>
-        <mesh filename="package://reemc_description/meshes/base/base.stl" />
+        <mesh filename="package://reemc_description/meshes/base/base.dae" />
       </geometry>
       <material name="LightGrey" />
@@ -27,5 +27,5 @@
       <origin xyz="-0.022 0 0.01" rpy="0 0 0" />
       <geometry>
-        <box size="0.27 0.295 0.14"/>
+        <box size="0.3 0.35 0.14"/>
       </geometry>
     </collision>
@@ -68,9 +68,9 @@
   <xacro:reemc_stereo_camera parent="head_2_link" name="stereo" focal_length="461.941850" hfov="${71.0*deg_to_rad}" image_format="B8G8R8" image_width="659" image_height="493">
 <!-- The following transformations expresses the pose of the stereo_link (X pointing forward, Z upwards and Y leftwards, contrary to the stereo_optical_link which has Z pointing forward) wrt  head_2_link. -->
-    <origin xyz="0.08203  -0.11558  0.0365" rpy="1.56293 -0.00855922 -0.0201307" />
+    <origin xyz="0.08203  -0.0935  0.0365" rpy="1.56293 -0.00855922 -0.0201307" />
   </xacro:reemc_stereo_camera>
   <xacro:reemc_back_camera parent="torso_2_link" name="back_camera" focal_length="376.003507" hfov="${89.999451423*deg_to_rad}" image_format="B8G8R8" image_width="752" image_height="480" >
     <!-- The following transformations expresses the pose of the back_camera_link (X pointing forward, Z upwards and Y leftwards, contrary to the stereo_optical_link which has Z pointing forward) wrt  torso_2_link. -->
-    <origin xyz="-0.09 -0.25 0" rpy="${-90.0*deg_to_rad} 0 ${180.0*deg_to_rad}" />
+    <origin xyz="-0.128 -0.317 0" rpy="${-90.0*deg_to_rad} 0 ${180.0*deg_to_rad}" />
   </xacro:reemc_back_camera>
   <!-- imu -->

File: reemc_common/reemc_description/urdf/arm/arm.urdf.xacro (robot description, xacro)
@@ -55,5 +55,5 @@
       <parent link="${parent}" />
       <child link="${name}_${side}_1_link" />
-      <origin xyz="0 -0.318 0" rpy="${(-165.0*reflect) * deg_to_rad} 0 0" />
+      <origin xyz="0 -0.31827 0" rpy="${(-165.0*reflect) * deg_to_rad} 0 0" />
       <axis xyz="0 0 1" />
       <limit lower="${-45.0 * deg_to_rad}" upper="${180.0 * deg_to_rad}" effort="${arm_1_max_effort}" velocity="${arm_1_max_vel}" />
@@ -90,5 +90,5 @@
       <parent link="${name}_${side}_1_link" />
       <child link="${name}_${side}_2_link" />
-      <origin xyz="0 0 ${0.2385 * reflect}" rpy="${-90.0 * reflect * deg_to_rad} ${-75.0 * reflect * deg_to_rad} ${90.0 * deg_to_rad}" />
+      <origin xyz="0 0 ${0.21749 * reflect}" rpy="${-90.0 * reflect * deg_to_rad} ${-75.0 * reflect * deg_to_rad} ${90.0 * deg_to_rad}" />
       <axis xyz="0 0 1" />
       <limit lower="${-15.0 * deg_to_rad}" upper="${120.0 * deg_to_rad}" effort="${arm_2_max_effort}" velocity="${arm_2_max_vel}" />

File: reemc_common/reemc_description/urdf/hand/hand.urdf.xacro (robot description, xacro)
@@ -33,7 +33,7 @@
     <link name="${hand_name}_${hand_side}_${finger_name}_link">
       <inertial>
-        <origin xyz="0 0 0" rpy="0 0 0" /> <!--TODO: Fill up-->
-        <mass value="0.05" />
-        <inertia ixx="0"  ixy="0"  ixz="0" iyy="0" iyz="0" izz="0" /> <!--TODO: Fill up-->
+        <origin xyz="0.00175 -0.01837 -0.00198" rpy="0 0 0" /> <!--TODO: Fill up-->
+        <mass value="0.055" />
+        <inertia ixx="0.00001450121"  ixy="-0.00000065488"  ixz="-0.00000039654" iyy="0.0000072995" iyz="0.00000012168" izz="0.00001262409" /> <!--TODO: Fill up-->
       </inertial>
       <visual>
@@ -69,7 +69,7 @@
     <link name="${hand_name}_${hand_side}_${finger_name}_1_link">
       <inertial>
-        <origin xyz="0 0 0" rpy="0 0 0" /> <!--TODO: Fill up-->
-        <mass value="0.05" />
-        <inertia ixx="0"  ixy="0"  ixz="0" iyy="0" iyz="0" izz="0" /> <!--TODO: Fill up-->
+        <origin xyz="0.00175 -0.01837 -0.00198" rpy="0 0 0" /> <!--TODO: Fill up-->
+        <mass value="0.055" />
+        <inertia ixx="0.00001450121"  ixy="-0.00000065488"  ixz="-0.00000039654" iyy="0.0000072995" iyz="0.00000012168" izz="0.00001262409" /> <!--TODO: Fill up-->
       </inertial>
       <visual>
@@ -97,7 +97,7 @@
     <link name="${hand_name}_${hand_side}_${finger_name}_2_link">
       <inertial>
-        <origin xyz="0 0 0" rpy="0 0 0" /> <!--TODO: Fill up-->
-        <mass value="0.05" />
-        <inertia ixx="0"  ixy="0"  ixz="0" iyy="0" iyz="0" izz="0" /> <!--TODO: Fill up-->
+        <origin xyz="0.00181 -0.01275 -0.00064" rpy="0 0 0" /> <!--TODO: Fill up-->
+        <mass value="0.02972" />
+        <inertia ixx="0.00000428193"  ixy="-0.00000049978"  ixz="-0.00000002985" iyy="0.00000254434" iyz="0.00000007762" izz="0.00000345152" /> <!--TODO: Fill up-->
       </inertial>
       <visual>
@@ -125,7 +125,7 @@
     <link name="${hand_name}_${hand_side}_${finger_name}_3_link">
       <inertial>
-        <origin xyz="0 0 0" rpy="0 0 0" /> <!--TODO: Fill up-->
-        <mass value="0.05" />
-        <inertia ixx="0"  ixy="0"  ixz="0" iyy="0" iyz="0" izz="0" /> <!--TODO: Fill up-->
+        <origin xyz="0 -0.00704 0.00019" rpy="0 0 0" /> <!--TODO: Fill up-->
+        <mass value="0.01522" />
+        <inertia ixx="0.00000128478"  ixy="-0.00000008056"  ixz="-0.00000001698" iyy="0.00000080139" iyz="-0.00000002884" izz="0.00000090928" /> <!--TODO: Fill up-->
       </inertial>
       <visual>
@@ -210,7 +210,7 @@
     <link name="${name}_${side}_thumb_link">
       <inertial>
-        <origin xyz="0 0 0" rpy="0 0 0" /> <!--TODO: Fill up-->
-        <mass value="0.05" />
-        <inertia ixx="0"  ixy="0"  ixz="0" iyy="0" iyz="0" izz="0" /> <!--TODO: Fill up-->
+        <origin xyz="0.00049 0.04179 0.00451" rpy="0 0 0" /> <!--TODO: Fill up-->
+        <mass value="0.07088" />
+        <inertia ixx="0.0000699364"  ixy="0.00000345915"  ixz="0.00000425008" iyy="0.00002675459" iyz="0.00002381865" izz="0.00004787167" /> <!--TODO: Fill up-->
       </inertial>
       <visual>

File: reemc_common/reemc_description/urdf/head/head.urdf.xacro (robot description, xacro)
@@ -23,19 +23,19 @@
     <link name="${name}_link">
       <inertial>
-        <origin xyz="0.01741 0.00466 -0.00434" rpy="0 0 0" />
-        <mass value="0.98547" />
+        <origin xyz="0.01819	0.00248	-0.00517" rpy="0 0 0" />
+        <mass value="1.11967" />
         <!-- NOTE: Assuming cylinder with r=0.06, h=0.08 -->
 <!--         <inertia ixx="0.0014125"  ixy="0"  ixz="0" iyy="0.0014125" iyz="0" izz="0.0017738" /> -->
-        <inertia ixx="0"  ixy="0"  ixz="0" iyy="0" iyz="0" izz="0" />
+        <inertia ixx="0.00111370229"  ixy="0.00003992198"  ixz="-0.00012464155" iyy="0.00111361487" iyz="0.00001943162" izz="0.00114794061" />
       </inertial>
       <visual>
         <origin rpy="0 0 0" xyz="-0.03 0 0"/> <!--TODO: Remove offset when good meshes arrive-->
         <geometry>
-          <mesh filename="package://reemc_description/meshes/head/head_1.stl" />
+          <mesh filename="package://reemc_description/meshes/head/head_1.dae" />
         </geometry>
         <material name="DarkGrey" />
       </visual>
       <collision>
-        <origin xyz="0 0 0" rpy="0 0 0" />
+        <origin xyz="-0.03 0 0" rpy="0 0 0" />
         <geometry>
           <mesh filename="package://reemc_description/meshes/head/head_1_collision.stl" />
@@ -46,5 +46,5 @@
       <parent link="${parent}"/>
       <child link="${name}_link"/>
-      <origin xyz="-0.024 -0.4 0" rpy="${90.0 * deg_to_rad} 0 0" />
+      <origin xyz="0.0 -0.42316 0" rpy="${90.0 * deg_to_rad} 0 0" />
       <axis xyz="0 0 1" />
       <limit lower="${-75.0 * deg_to_rad}" upper="${75.0 * deg_to_rad}" effort="3.4" velocity="${head_max_vel}" />
@@ -71,20 +71,20 @@
     <link name="${name}_link">
       <inertial>
-        <origin xyz="-0.04431 -0.13008 0.00011" rpy="0 0 0" />
-        <mass value="1.20862" />
+        <origin xyz="0.01183 -0.08098 0.00104" rpy="0 0 0" />
+        <mass value="1.63134" />
         <!-- NOTE: Assuming box with d=0.28433, w=0.20302, h=0.26741 -->
 <!--         <inertia ixx="0.011353"  ixy="0"  ixz="0" iyy="0.012294" iyz="0" izz="0.015345" /> -->
         <!--NOTE: Low (0.1 or lower) diagonal inertia values make Gazebo 1.0.2 simulation unstable when head sensors are added.-->
-        <inertia ixx="0.25"  ixy="0"  ixz="0" iyy="0.25" iyz="0" izz="0.25" />
+        <inertia ixx="0.00640199093"  ixy="0.00012197067"  ixz="-0.00000897011" iyy="0.00676228591" iyz="-0.0000552329" izz="0.00614192438" />
       </inertial>
       <visual>
         <origin rpy="0 0 0" xyz="-0.03 0 0"/> <!--TODO: Remove offset when good meshes arrive-->
         <geometry>
-          <mesh filename="package://reemc_description/meshes/head/head_2.stl" />
+          <mesh filename="package://reemc_description/meshes/head/head_2.dae" />
         </geometry>
         <material name="LightGrey" />
       </visual>
       <collision>
-        <origin xyz="0 0 0" rpy="0 0 0" />
+        <origin xyz="-0.03 0 0" rpy="0 0 0" />
         <geometry>
           <mesh filename="package://reemc_description/meshes/head/head_2_collision.stl" />

File: reemc_common/reemc_description/urdf/leg/leg.urdf.xacro (robot description, xacro)
@@ -40,5 +40,5 @@
         <origin rpy="0 0 0" xyz="0 0 0"/>
         <geometry>
-          <mesh filename="package://reemc_description/meshes/leg/leg_1.stl" scale="1 1 1"/>
+          <mesh filename="package://reemc_description/meshes/leg/leg_1.dae" scale="1 1 1"/>
         </geometry>
         <material name="LightGrey" />
@@ -46,14 +46,14 @@
       </link>
     <joint name="leg_${side}_1_joint" type="revolute">
-        <origin  xyz="0  ${-reflect*0.075} -0.139" rpy="0 0 0"/>
+        <origin  xyz="0  ${-reflect*0.075} -0.14353" rpy="0 0 0"/>
         <axis xyz="0 0 1"/>
         <parent link="${parent}"/>
         <child link="leg_${side}_1_link"/>
         <dynamics friction="${leg_friction}" damping="${leg_damping}"/>
-        <limit lower="${-45 * deg_to_rad}" upper="${30.0 * deg_to_rad}" effort="${leg_1_joint_effort}" velocity="${leg_1_joint_max_vel}" />
+        <limit lower="${-37.5*deg_to_rad + reflect*7.5*deg_to_rad}" upper="${37.5*deg_to_rad + reflect*7.5*deg_to_rad}" effort="${leg_1_joint_effort}" velocity="${leg_1_joint_max_vel}" />
         <safety_controller k_position="100"
                            k_velocity="100"
-                           soft_lower_limit="${-45.0 * deg_to_rad + leg_eps}"
-                           soft_upper_limit="${ 30.0 * deg_to_rad - leg_eps}" />
+                           soft_lower_limit="${-37.5*deg_to_rad + reflect*7.5*deg_to_rad + leg_eps}"
+                           soft_upper_limit="${ 37.5*deg_to_rad + reflect*7.5*deg_to_rad - leg_eps}" />
       </joint>
       <link name="leg_${side}_2_link">
@@ -77,9 +77,9 @@
         <child link="leg_${side}_2_link"/>
         <dynamics friction="${leg_friction}" damping="${leg_damping}"/>
-        <limit lower="${-22.5 * deg_to_rad - reflect*7.5*deg_to_rad}" upper="${22.5 * deg_to_rad - reflect*7.5*deg_to_rad}" effort="${leg_2_joint_effort}" velocity="${leg_2_joint_max_vel}" />
+        <limit lower="${-22.5*deg_to_rad - reflect*7.5*deg_to_rad}" upper="${22.5*deg_to_rad - reflect*7.5*deg_to_rad}" effort="${leg_2_joint_effort}" velocity="${leg_2_joint_max_vel}" />
         <safety_controller k_position="100"
                            k_velocity="100"
-                           soft_lower_limit="${-22.5 * deg_to_rad - reflect*7.5*deg_to_rad + leg_eps}"
-                           soft_upper_limit="${ 22.5 * deg_to_rad - reflect*7.5*deg_to_rad - leg_eps}" />
+                           soft_lower_limit="${-22.5*deg_to_rad - reflect*7.5*deg_to_rad + leg_eps}"
+                           soft_upper_limit="${ 22.5*deg_to_rad - reflect*7.5*deg_to_rad - leg_eps}" />
     </joint>
     <link name="leg_${side}_3_link">
@@ -90,7 +90,7 @@
       </inertial>
      <visual>
-        <origin rpy="${180.0* deg_to_rad} 0 0" xyz="0 0 0"/>
-        <geometry>
-          <mesh filename="package://reemc_description/meshes/leg/leg_3.stl" scale="1 1 ${-1*reflect}"/>
+        <origin rpy="0 0 0" xyz="0 0 0"/>
+        <geometry>
+          <mesh filename="package://reemc_description/meshes/leg/leg_3.dae" scale="1 1 ${-1*reflect}"/>
         </geometry>
         <material name="LightGrey" />
@@ -124,5 +124,5 @@
         <origin rpy="0 0 0" xyz="0 0 0"/>
         <geometry>
-          <mesh filename="package://reemc_description/meshes/leg/leg_4.stl" scale="1 1 ${-1*reflect}"/>
+          <mesh filename="package://reemc_description/meshes/leg/leg_4.dae" scale="1 1 ${-1*reflect}"/>
         </geometry>
         <material name="LightGrey" />
@@ -181,7 +181,7 @@
       </inertial>
       <visual>
-        <origin rpy="0 ${-90.0*deg_to_rad} 0" xyz="0.110 0 0"/>
-        <geometry>
-          <mesh filename="package://reemc_description/meshes/leg/sole.stl" scale="1 ${-1*reflect} 1"/>
+        <origin rpy="0 0 0" xyz="0 0 0"/>
+        <geometry>
+          <mesh filename="package://reemc_description/meshes/leg/leg_6.dae" scale="1 ${-1*reflect} 1"/>
         </geometry>
         <material name="LightGrey" />
@@ -200,9 +200,9 @@
       <child link="leg_${side}_6_link"/>
       <dynamics friction="${leg_friction}" damping="${leg_damping}"/>
-      <limit lower="${-15 * deg_to_rad}" upper="${ 30.0 * deg_to_rad}" effort="${leg_6_joint_effort}" velocity="${leg_6_joint_max_vel}" />
-      <safety_controller k_position="100"
-                         k_velocity="100"
-                         soft_lower_limit="${-15.0 * deg_to_rad + leg_eps}"
-                         soft_upper_limit="${ 30.0 * deg_to_rad - leg_eps}" />
+      <limit lower="${-22.5*deg_to_rad + reflect*7.5*deg_to_rad}" upper="${ 22.5*deg_to_rad + reflect*7.5*deg_to_rad}" effort="${leg_6_joint_effort}" velocity="${leg_6_joint_max_vel}" />
+      <safety_controller k_position="100"
+                         k_velocity="100"
+                         soft_lower_limit="${-22.5*deg_to_rad + reflect*7.5*deg_to_rad + leg_eps}"
+                         soft_upper_limit="${ 22.5*deg_to_rad + reflect*7.5*deg_to_rad - leg_eps}" />
     </joint>
     <link name="${side}_sole_link">
@@ -280,6 +280,6 @@
     <xacro:reemc_leg_simple_transmission name="${name}" side="${side}" number="5" reduction="${leg_reduction}" />
     <xacro:reemc_leg_simple_transmission name="${name}" side="${side}" number="6" reduction="${leg_reduction}" />
-   <xacro:reemc_laser name="${side}_laser" parent="leg_${side}_6_link" ros_topic="${side}_scan" update_rate="10.0" min_angle="${-90*deg_to_rad}" max_angle="${90*deg_to_rad}" nrays="360" >
-      <origin xyz="0.07 ${0.071 -((1+reflect)*0.01 + 0.061)} ${0.170 -0.085}" rpy="0 ${-90.0*deg_to_rad} 0" />
+   <xacro:reemc_laser name="${side}_laser" parent="${side}_sole_link" ros_topic="${side}_scan" update_rate="10.0" min_angle="${-90*deg_to_rad}" max_angle="${90*deg_to_rad}" nrays="360" >
+     <origin xyz="${0.170 -0.085} ${0.071 -((1+reflect)*0.01 + 0.061)} ${0.04}" rpy="0.0 0.0 ${-30.0*reflect*deg_to_rad}" />
     </xacro:reemc_laser>
   </xacro:macro>

File: reemc_common/reemc_description/urdf/sensors/mvbluefox_back_camera.gazebo.xacro (robot description, xacro)
@@ -30,5 +30,5 @@
          <alwaysOn>true</alwaysOn>
          <updateRate>15.0</updateRate>
-         <cameraName>/reemc/${name}</cameraName>
+         <cameraName>${name}</cameraName>
          <imageTopicName>image</imageTopicName>
          <cameraInfoTopicName>camera_info</cameraInfoTopicName>

File: reemc_common/reemc_description/urdf/sensors/prosilica_stereo_camera.gazebo.xacro (robot description, xacro)
@@ -40,5 +40,5 @@
          <alwaysOn>true</alwaysOn>
          <updateRate>25.0</updateRate>
-         <cameraName>/reemc/${name}</cameraName>
+         <cameraName>${name}</cameraName>
          <imageTopicName>image</imageTopicName>
          <cameraInfoTopicName>camera_info</cameraInfoTopicName>

File: reemc_common/reemc_description/urdf/torso/torso.urdf.xacro (robot description, xacro)
@@ -37,5 +37,5 @@
       <parent link="${parent}"/>
       <child link="${name}_1_link"/>
-      <origin xyz="0 0 0.139" rpy="0 0 0" />
+      <origin xyz="0 0 0.14353" rpy="0 0 0" />
       <axis xyz="0 0 1" />
       <limit lower="${-75.0 * deg_to_rad}" upper="${75.0 * deg_to_rad}" effort="${torso_max_effort}" velocity="${torso_max_vel}" />
@@ -59,5 +59,5 @@
         <origin rpy="0 0 0" xyz="0 0 0"/>
         <geometry>
-          <mesh filename="package://reemc_description/meshes/torso/torso_2.stl" />
+          <mesh filename="package://reemc_description/meshes/torso/torso_2.dae" />
         </geometry>
         <material name="LightGrey" />
